File: tests/demo/synthetic_electrical_connectivity_demo.kicad_pcb (KiCad board)
At the start: 3 copper layers, 116 x 72 mm, 8 parts

Commit message: fix(demo): declare a valid copper layer count
Other:
- copper layers 3 -> 4
Changed lines of the file:
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@@
 		(0 "F.Cu" signal)
 		(4 "In1.Cu" signal)
+		(6 "In2.Cu" signal)
 		(2 "B.Cu" signal)
 		(5 "F.SilkS" user "F.Silkscreen")
